File: pcb/channel/oscillator.sch (KiCad schematic (older format))
At the start: 36 parts, among them IC6 MCP6542-E_MS, IC7 MCP6074-E_ST, IC8 MCP6541T-I_OT, Q1 NX3008NBKW,115, Q2 MBT3904DW1, Q3 MMBT3904

Commit message: Set final resistor values for oscillator
Parts:
- R23, R24: value 1 -> 90.1k
- R27: value 1 -> 10k
- R8: value 4.7k -> 1k
Changed lines of the file:
@@
 P 6750 4950
 F 0 "R23" V 6550 4950 50  0000 C CNN
-F 1 "1" V 6650 4950 50  0000 C CNN
+F 1 "90.1k" V 6650 4950 50  0000 C CNN
 F 2 "Resistor_SMD:R_0603_1608Metric_Pad1.05x0.95mm_HandSolder" V 6680 4950 50  0001 C CNN
 F 3 "~" H 6750 4950 50  0001 C CNN
@@
 P 6750 5100
 F 0 "R24" V 6850 5100 50  0000 C CNN
-F 1 "1" V 6950 5100 50  0000 C CNN
+F 1 "90.1k" V 6950 5100 50  0000 C CNN
 F 2 "Resistor_SMD:R_0603_1608Metric_Pad1.05x0.95mm_HandSolder" V 6680 5100 50  0001 C CNN
 F 3 "~" H 6750 5100 50  0001 C CNN
@@
 P 7150 4950
 F 0 "R27" V 6950 4950 50  0000 C CNN
-F 1 "1" V 7050 4950 50  0000 C CNN
+F 1 "10k" V 7050 4950 50  0000 C CNN
 F 2 "Resistor_SMD:R_0603_1608Metric_Pad1.05x0.95mm_HandSolder" V 7080 4950 50  0001 C CNN
 F 3 "~" H 7150 4950 50  0001 C CNN
@@
 P 2950 4250
 F 0 "R8" H 2750 4300 50  0000 L CNN
-F 1 "4.7k" H 2700 4200 50  0000 L CNN
+F 1 "1k" H 2750 4200 50  0000 L CNN
 F 2 "Resistor_SMD:R_0603_1608Metric_Pad1.05x0.95mm_HandSolder" V 2880 4250 50  0001 C CNN
 F 3 "~" H 2950 4250 50  0001 C CNN
