File: pcb/channel/channel.kicad_pcb (KiCad board)
At the start: 2 copper layers, 104.9 x 32.6 mm, 199 parts, among them IC10 DMC2700UDM-7, IC11 MCP6074-E_ST, IC12 MCP6074-E_ST, IC13 MCP6074-E_ST, IC14 DMC2700UDM-7, IC15 DMC2700UDM-7, IC16 DMC2700UDM-7, IC2 MCP47CVB22-E_UN, IC3 MCP6074-E_ST, IC4 MCP6072-E_SN, IC5 DAC5574IDGS, IC6 MCP6542-E_MS, IC7 MCP6074-E_ST, IC8 MCP6541T-I_OT, IC9 MCP6074-E_ST, J1 Conn_02x02_Odd_Even, J10 Conn_02x03_Odd_Even, J11 Conn_01x08_Male, J2 Conn_02x04_Odd_Even, J3 Conn_01x06_Male, J4 Conn_01x02, J5 Conn_01x08_Male, J6 Conn_01x02, J7 Conn_01x02, J8 Conn_02x03_Odd_Even, J9 Conn_02x03_Odd_Even, Q1 NX3008NBKW,115, Q10 MBT3946DW1T1, Q11 MBT3946DW1T1, Q12 MBT3946DW1T1, Q13 2SK2145-BL_TE85L,F, Q14 2SK2145-BL_TE85L,F, Q15 2SK3557-7-TB-E, Q16 2SK3557-7-TB-E, Q17 2SK3557-7-TB-E, Q18 NX3008PBKW,115, Q2 MBT3904DW1, Q3 MMBT3904, Q4 MBT3946DW1T1, Q5 MBT3946DW1T1, Q6 MBT3946DW1T1, Q7 MBT3946DW1T1, Q8 MBT3946DW1T1, Q9 MBT3946DW1T1

Commit message: Rename/renumbering (I think)
Parts:
- R107, R108, R113, R114, R119, R120: value 1Meg -> 100k
- R23, R24: value 1 -> 90.1k
- R27: value 1 -> 10k
- R32: value 82k -> 21.5k
- R34: value 10k -> 13.3k
- R35: value 180k -> 68.1k
- R46: value 2k -> 3k
- R8: value 4.7k -> 1k
Connections:
- net FSEL1 renamed FSELA
- net FSEL2 renamed FSELB
- net OSEL1 renamed OSELA
- net OSEL2 renamed OSELB
- IC2 pad 3: (no net) -> Net-(IC2-Pad3)
- J2 pad 2: /Switch4 (3.3V)/SIGNAL2 -> /Switch4 (3.3V)/SIGNAL4
- J2 pad 4: /Switch4 (3.3V)/SIGNAL1 -> /Switch4 (3.3V)/SIGNAL3
- J2 pad 6: /Switch4 (3.3V)/SIGNAL4 -> /Switch4 (3.3V)/SIGNAL2
- J2 pad 8: /Switch4 (3.3V)/SIGNAL3 -> /Switch4 (3.3V)/SIGNAL1
- Q11 pad 1: /Switch4 (3.3V)/SIGNAL2 -> /Switch4 (3.3V)/SIGNAL4
- Q11 pad 4: /Switch4 (3.3V)/SIGNAL2 -> /Switch4 (3.3V)/SIGNAL4
- Q12 pad 1: /Switch4 (3.3V)/SIGNAL1 -> /Switch4 (3.3V)/SIGNAL3
- Q12 pad 4: /Switch4 (3.3V)/SIGNAL1 -> /Switch4 (3.3V)/SIGNAL3
- Q8 pad 1: /Switch4 (3.3V)/SIGNAL4 -> /Switch4 (3.3V)/SIGNAL2
- Q8 pad 4: /Switch4 (3.3V)/SIGNAL4 -> /Switch4 (3.3V)/SIGNAL2
- Q9 pad 1: /Switch4 (3.3V)/SIGNAL3 -> /Switch4 (3.3V)/SIGNAL1
- Q9 pad 4: /Switch4 (3.3V)/SIGNAL3 -> /Switch4 (3.3V)/SIGNAL1
Routing:
- net /Switch4 (3.3V)/SIGNAL3: track 14.7 -> 12.7 mm
- net /Switch4 (3.3V)/SIGNAL1: track 12.7 -> 14.7 mm
- net /Switch4 (3.3V)/SIGNAL4: track 11.6 -> 10.4 mm
- net /Switch4 (3.3V)/SIGNAL2: track 10.4 -> 11.6 mm
