File: pcb/channel/switch2_unbuf_0.1v.sch (KiCad schematic (older format))
At the start: 2 parts, among them IC14 DMC2700UDM-7

Commit message: Rename/renumbering (I think)
Changed lines of the file:
@@
 $Descr A4 11693 8268
 encoding utf-8
-Sheet 14 19
+Sheet 10 19
 Title ""
 Date ""
@@
 AR Path="/604FDE2C/6050367E/604E80E2" Ref="IC16"  Part="1"
 AR Path="/6048E07A/6055BEFE/604E80E2" Ref="IC10"  Part="1"
-F 0 "IC16" H 5750 4415 50  0000 C CNN
+F 0 "IC10" H 5750 4415 50  0000 C CNN
 F 1 "DMC2700UDM-7" H 5750 4324 50  0000 C CNN
 F 2 "footprints:SOT95P285X140-6N" H 6050 4250 50  0001 L CNN
@@
 AR Path="/604FDE2C/6050367E/604F252B" Ref="R127"  Part="1"
 AR Path="/6048E07A/6055BEFE/604F252B" Ref="R77"  Part="1"
-F 0 "R127" V 4743 4150 50  0000 C CNN
+F 0 "R77" V 4743 4150 50  0000 C CNN
 F 1 "4.7k" V 4834 4150 50  0000 C CNN
 F 2 "Resistor_SMD:R_0603_1608Metric_Pad1.05x0.95mm_HandSolder" V 4880 4150 50  0001 C CNN
