File: pcb/channel/switch2_unbuf_3.3v.sch (KiCad schematic (older format))
At the start: 11 parts, among them Q4 MBT3946DW1T1, Q5 MBT3946DW1T1, Q6 MBT3946DW1T1

Commit message: Rename/renumbering (I think)
Changed lines of the file:
@@
 $Descr A4 11693 8268
 encoding utf-8
-Sheet 8 19
+Sheet 7 19
 Title ""
 Date ""
@@
 AR Path="/603FA658/6043E0DE/6040107D" Ref="Q?"  Part="1"
 AR Path="/603FA658/6045F739/6040107D" Ref="Q8"  Part="2"
-F 0 "Q8" H 5800 3250 50  0000 L CNN
+F 0 "Q5" H 5800 3250 50  0000 L CNN
 F 1 "MBT3946DW1T1" H 5450 3150 50  0000 L CNN
 F 2 "Package_TO_SOT_SMD:SOT-363_SC-70-6" H 6150 3500 50  0001 C CNN
@@
 AR Path="/603FA658/6043E0DE/60401083" Ref="Q?"  Part="2"
 AR Path="/603FA658/6045F739/60401083" Ref="Q8"  Part="1"
-F 0 "Q8" H 6200 3250 50  0000 L CNN
+F 0 "Q5" H 6200 3250 50  0000 L CNN
 F 1 "MBT3946DW1T1" H 5850 3150 50  0000 L CNN
 F 2 "Package_TO_SOT_SMD:SOT-363_SC-70-6" H 6550 3500 50  0001 C CNN
@@
 AR Path="/603FA658/6043E0DE/60420711" Ref="R?"  Part="1"
 AR Path="/603FA658/6045F739/60420711" Ref="R59"  Part="1"
-F 0 "R59" V 4593 3100 50  0000 C CNN
+F 0 "R51" V 4593 3100 50  0000 C CNN
 F 1 "100k" V 4684 3100 50  0000 C CNN
 F 2 "Resistor_SMD:R_0603_1608Metric_Pad1.05x0.95mm_HandSolder" V 4730 3100 50  0001 C CNN
@@
 AR Path="/603FA658/6043E0DE/60422A4C" Ref="R?"  Part="1"
 AR Path="/603FA658/6045F739/60422A4C" Ref="R61"  Part="1"
-F 0 "R61" H 5100 3700 50  0000 L CNN
+F 0 "R53" H 5100 3700 50  0000 L CNN
 F 1 "100k" H 5050 3600 50  0000 L CNN
 F 2 "Resistor_SMD:R_0603_1608Metric_Pad1.05x0.95mm_HandSolder" V 5230 3650 50  0001 C CNN
@@
 AR Path="/603FA658/6043E0DE/60425F9E" Ref="R?"  Part="1"
 AR Path="/603FA658/6045F739/60425F9E" Ref="R63"  Part="1"
-F 0 "R63" V 5343 3400 50  0000 C CNN
+F 0 "R55" V 5343 3400 50  0000 C CNN
 F 1 "100k" V 5434 3400 50  0000 C CNN
 F 2 "Resistor_SMD:R_0603_1608Metric_Pad1.05x0.95mm_HandSolder" V 5480 3400 50  0001 C CNN
@@
 AR Path="/603FA658/6043E0DE/6042EBB1" Ref="R?"  Part="1"
 AR Path="/603FA658/6045F739/6042EBB1" Ref="R65"  Part="1"
-F 0 "R65" V 6543 3400 50  0000 C CNN
+F 0 "R57" V 6543 3400 50  0000 C CNN
 F 1 "100k" V 6634 3400 50  0000 C CNN
 F 2 "Resistor_SMD:R_0603_1608Metric_Pad1.05x0.95mm_HandSolder" V 6680 3400 50  0001 C CNN
@@
 AR Path="/603FA658/6043E0DE/603FCA89" Ref="Q?"  Part="1"
 AR Path="/603FA658/6045F739/603FCA89" Ref="Q9"  Part="1"
-F 0 "Q9" H 5850 4750 50  0000 L CNN
+F 0 "Q6" H 5850 4750 50  0000 L CNN
 F 1 "MBT3946DW1T1" H 5450 4650 50  0000 L CNN
 F 2 "Package_TO_SOT_SMD:SOT-363_SC-70-6" H 6150 5000 50  0001 C CNN
@@
 AR Path="/603FA658/6043E0DE/603FD889" Ref="Q?"  Part="2"
 AR Path="/603FA658/6045F739/603FD889" Ref="Q9"  Part="2"
-F 0 "Q9" H 6200 4750 50  0000 L CNN
+F 0 "Q6" H 6200 4750 50  0000 L CNN
 F 1 "MBT3946DW1T1" H 5800 4650 50  0000 L CNN
 F 2 "Package_TO_SOT_SMD:SOT-363_SC-70-6" H 6550 5000 50  0001 C CNN
@@
 AR Path="/603FA658/6043E0DE/603FFB63" Ref="Q?"  Part="1"
 AR Path="/603FA658/6045F739/603FFB63" Ref="Q7"  Part="1"
-F 0 "Q7" H 5050 5050 50  0000 L CNN
+F 0 "Q4" H 5050 5050 50  0000 L CNN
 F 1 "MBT3946DW1T1" H 4700 4950 50  0000 L CNN
 F 2 "Package_TO_SOT_SMD:SOT-363_SC-70-6" H 5400 5300 50  0001 C CNN
@@
 AR Path="/603FA658/6043E0DE/60401504" Ref="R?"  Part="1"
 AR Path="/603FA658/6045F739/60401504" Ref="R60"  Part="1"
-F 0 "R60" V 4593 5200 50  0000 C CNN
+F 0 "R52" V 4593 5200 50  0000 C CNN
 F 1 "100k" V 4684 5200 50  0000 C CNN
 F 2 "Resistor_SMD:R_0603_1608Metric_Pad1.05x0.95mm_HandSolder" V 4730 5200 50  0001 C CNN
@@
 AR Path="/603FA658/6043E0DE/60403872" Ref="R?"  Part="1"
 AR Path="/603FA658/6045F739/60403872" Ref="R62"  Part="1"
-F 0 "R62" H 5100 4700 50  0000 L CNN
+F 0 "R54" H 5100 4700 50  0000 L CNN
 F 1 "100k" H 5050 4600 50  0000 L CNN
 F 2 "Resistor_SMD:R_0603_1608Metric_Pad1.05x0.95mm_HandSolder" V 5230 4650 50  0001 C CNN
@@
 AR Path="/603FA658/6043E0DE/6040866B" Ref="R?"  Part="1"
 AR Path="/603FA658/6045F739/6040866B" Ref="R64"  Part="1"
-F 0 "R64" V 5343 4900 50  0000 C CNN
+F 0 "R56" V 5343 4900 50  0000 C CNN
 F 1 "100k" V 5434 4900 50  0000 C CNN
 F 2 "Resistor_SMD:R_0603_1608Metric_Pad1.05x0.95mm_HandSolder" V 5480 4900 50  0001 C CNN
@@
 AR Path="/603FA658/6043E0DE/604173A7" Ref="R?"  Part="1"
 AR Path="/603FA658/6045F739/604173A7" Ref="R66"  Part="1"
-F 0 "R66" V 6543 4900 50  0000 C CNN
+F 0 "R58" V 6543 4900 50  0000 C CNN
 F 1 "100k" V 6634 4900 50  0000 C CNN
 F 2 "Resistor_SMD:R_0603_1608Metric_Pad1.05x0.95mm_HandSolder" V 6680 4900 50  0001 C CNN
@@
 AR Path="/603FA658/6043E0DE/603FFB69" Ref="Q?"  Part="2"
 AR Path="/603FA658/6045F739/603FFB69" Ref="Q7"  Part="2"
-F 0 "Q7" H 5050 3250 50  0000 L CNN
+F 0 "Q4" H 5050 3250 50  0000 L CNN
 F 1 "MBT3946DW1T1" H 4700 3350 50  0000 L CNN
 F 2 "Package_TO_SOT_SMD:SOT-363_SC-70-6" H 5400 3200 50  0001 C CNN
